Commit message: fixes

File: revolt_gazebosim/urdf/revolt_gazebosim.xacro (robot description, xacro)
@@ -2,46 +2,6 @@
 <robot xmlns:xacro="http://www.ros.org/wiki/xacro" name="revolt">
   <xacro:include filename="$(find revolt_description)/urdf/revolt.urdf.xacro"/>
-   <xacro:if value="$(arg use_gazebo_ros_control)">
-    <ros2_control name="diff_controller" type="system">
-    <hardware>
-      <plugin>gazebo_ros2_control/GazeboSystem</plugin>
-    </hardware>
-    <joint name="left_wheel_joint">
-      <command_interface name="velocity">
-        <param name="min">-5</param>
-        <param name="max">5</param>
-      </command_interface>
-      <state_interface name="velocity"/>
-      <state_interface name="position"/>
-    </joint>
-    <joint name="right_wheel_joint">
-      <command_interface name="velocity">
-        <param name="min">-5</param>
-        <param name="max">5</param>
-      </command_interface>
-      <state_interface name="velocity"/>
-      <state_interface name="position"/>
-    </joint>
-  </ros2_control>
-    <gazebo>
-      <plugin filename="libgazebo_ros2_control.so" name="gazebo_ros2_control">
-          <parameters>$(find revolt_control)/config/revolt_controllers.yaml</parameters>
-      </plugin>
-      <plugin name="revolt_joint_state_caster" filename="libgazebo_ros_joint_state_publisher.so">
-      <ros>
-        <remapping>~/out:=joint_states</remapping>
-        <remapping>/tf:=tf</remapping>
-      </ros>
-      <update_rate>30</update_rate>
-      <joint_name>frontcaster_rotation_joint</joint_name>
-      <joint_name>frontcaster_wheel_joint</joint_name>
-      <joint_name>backcaster_rotation_joint</joint_name>
-      <joint_name>backcaster_wheel_joint</joint_name>
-    </plugin>
-    </gazebo>
-  </xacro:if>
-  <xacro:unless value="$(arg use_gazebo_ros_control)">
 	  <gazebo>
-    <plugin name="revolt_joint_state" filename="libgazebo_ros_joint_state_publisher.so">
+    <!-- <plugin name="revolt_joint_state" filename="libgazebo_ros_joint_state_publisher.so">
       <ros>
         <remapping>~/out:=joint_states</remapping>
@@ -55,10 +15,15 @@
       <joint_name>backcaster_rotation_joint</joint_name>
       <joint_name>backcaster_wheel_joint</joint_name>
+    </plugin> -->
+    <plugin filename="gz-sim-joint-state-publisher-system" name="gz::sim::systems::JointStatePublisher">
+      <topic>joint_states</topic> <!--from <ros><remapping> -->
+      <joint_name>right_wheel_joint</joint_name>
+      <joint_name>left_wheel_joint</joint_name>
+      <joint_name>frontcaster_rotation_joint</joint_name>
+      <joint_name>frontcaster_wheel_joint</joint_name>
+      <joint_name>backcaster_rotation_joint</joint_name>
+      <joint_name>backcaster_wheel_joint</joint_name>
     </plugin>
-    <plugin name='revolt_diff_drive' filename='libgazebo_ros_diff_drive.so'>
-      <ros>
-        <remapping>odom:=odom</remapping>
-        <remapping>/tf:=tf</remapping>
-      </ros>
+    <plugin filename="gz-sim-diff-drive-system" name="gz::sim::systems::DiffDrive">
       <!-- wheels -->
       <left_joint>left_wheel_joint</left_joint>
@@ -66,17 +31,16 @@
       <!-- kinematics -->
       <wheel_separation>0.187</wheel_separation>
-      <wheel_diameter>0.0757664</wheel_diameter>
+      <wheel_radius>0.038</wheel_radius>
       <!-- limits -->
-      <max_wheel_torque>20</max_wheel_torque>
-      <max_wheel_acceleration>1</max_wheel_acceleration>
-      <!-- output -->
-      <publish_odom>true</publish_odom>
-      <publish_odom_tf>true</publish_odom_tf>
-      <odometry_frame>odom</odometry_frame>
-      <robot_base_frame>base_footprint</robot_base_frame>
+      <max_linear_acceleration>0.033</max_linear_acceleration> <!-- computed from <max_linear_acceleration> in the original plugin-->
+      <topic>cmd_vel</topic> <!-- from <commant_topic> -->
+      <odom_topic>odom</odom_topic> <!-- from <odometry_topic> -->
+      <frame_id>odom</frame_id> <!-- from <odometry_frame> -->
+      <child_frame_id>base_footprint</child_frame_id> <!-- from <robot_base_frame> -->
+      <odom_publisher_frequency>30</odom_publisher_frequency> <!-- from <update_rate>-->
+      <tf_topic>/tf</tf_topic> <!-- Short topic name for tf output -->
     </plugin>
 	  </gazebo>
-  </xacro:unless>
-    <gazebo reference="rplidar_laser_link">
+    <!-- <gazebo reference="rplidar_laser_link">
       <sensor name="laser" type="ray">
         <ray>
@@ -141,4 +105,4 @@
           </plugin>
         </sensor>
-  </gazebo>
+  </gazebo> -->
 </robot>
