Commit message: Added gazebo plugins

File: revolt_description/urdf/revolt.urdf.xacro (robot description, xacro)
@@ -130,5 +130,5 @@
         </visual>
     </link>
-    <joint name="camera_mount" type="fixed">
+    <joint name="camera_mount_joint" type="fixed">
         <origin xyz="-0.099030762113532788682 -2.0560008597292656995e-11 0.094246835314834839781"
             rpy="1.570796326794896558 -2.0033280460268570124e-25 2.4319171023353502458e-16" />

File: revolt_gazebosim/urdf/revolt_gazebosim.xacro (robot description, xacro)
@@ -42,13 +42,16 @@
     </plugin>
 	  </gazebo>
-    <!-- <gazebo reference="rplidar_laser_link">
-      <sensor name="laser" type="ray">
-        <ray>
+<!--
+    <gazebo reference="rplidar_laser_link">
+      <sensor name="laser" type="gpu_lidar">
+        <visualize>false</visualize>
+        <update_rate>10</update_rate>
+        <lidar>
           <scan>
             <horizontal>
             <samples>720</samples>
             <resolution>1</resolution>
-            <min_angle>-3.14159265</min_angle>
-            <max_angle>3.14159265</max_angle>
+            <min_angle>-3.14</min_angle>
+            <max_angle>3.14</max_angle>
             </horizontal>
           </scan>
@@ -58,22 +61,73 @@
             <resolution>0.01</resolution>
           </range>
-          <noise>
-          <type>gaussian</type>
-          <mean>0.0</mean>
-          <stddev>0.01</stddev>
-        </noise>
-        </ray>
-        <always_on>true</always_on>
-        <visualize>true</visualize>
-        <update_rate>20.0</update_rate>
-        <plugin name="laser_controller" filename="libgazebo_ros_ray_sensor.so">
-          <ros>
-            <remapping>~/out:=scan</remapping>
-          </ros>
-          <frame_name>rplidar_laser_link</frame_name>
-          <output_type>sensor_msgs/LaserScan</output_type>
-        </plugin>
+        </lidar>
+        <topic>scan</topic>
+        <gz_frame_id>rplidar_laser_link</gz_frame_id>
       </sensor>
+    </gazebo> -->
+    <gazebo reference="rplidar_laser_link">
+        <sensor name="gpu_lidar" type="gpu_lidar">
+          <always_on>true</always_on>
+          <visualize>true</visualize>
+          <update_rate>5</update_rate>
+          <topic>scan</topic>
+          <gz_frame_id>base_scan</gz_frame_id>
+          <lidar>
+              <scan>
+                  <horizontal>
+                      <samples>360</samples>
+                      <resolution>1</resolution>
+                      <min_angle>-3.14</min_angle>
+                      <max_angle>3.14</max_angle>
+                  </horizontal>
+              </scan>
+              <range>
+                  <min>0.10</min>
+                  <max>12.0</max>
+                  <resolution>0.01</resolution>
+              </range>
+              <noise>
+                  <type>gaussian</type>
+                  <mean>0.0</mean>
+                  <stddev>0.001</stddev>
+              </noise>
+          </lidar>
+        </sensor>
     </gazebo>
+        <!-- <sensor name="gpu_lidar" type="gpu_lidar">
+          <always_on>true</always_on>
+          <visualize>true</visualize>
+          <pose>-0.064 0 0.121 0 0 0</pose>
+          <update_rate>5</update_rate>
+          <topic>scan</topic>
+          <gz_frame_id>base_scan</gz_frame_id>
+          <lidar>
+              <scan>
+                  <horizontal>
+                      <samples>360</samples>
+                      <resolution>1</resolution>
+                      <min_angle>-3.14</min_angle>
+                      <max_angle>3.14</max_angle>
+                  </horizontal>
+              </scan>
+              <range>
+                  <min>0.10</min>
+                  <max>12.0</max>
+                  <resolution>0.01</resolution>
+              </range>
+              <noise>
+                  <type>gaussian</type>
+                  <mean>0.0</mean>
+                  <stddev>0.001</stddev>
+              </noise>
+          </lidar>
+        </sensor> -->
+    <!-- <joint name="camera_optical_joint" type="fixed">
+        <parent link="camera_link"/>
+        <child link="camera_link_optical"/>
+        <origin xyz="0 0 0" rpy="0 0 0"/>
+        <axis xyz="0 0 0" />
+    </joint>
+    <link name="camera_link_optical"></link>
     <gazebo reference="camera_link">
         <sensor name='camera' type='camera'>
@@ -91,17 +145,6 @@
           <always_on>1</always_on>
           <update_rate>30</update_rate>
-          <plugin name='camera_controller' filename='libgazebo_ros_camera.so'>
-            <alwaysOn>1</alwaysOn>
-            <cameraName>camera</cameraName>
-            <imageTopicName>image_raw</imageTopicName>
-            <cameraInfoTopicName>camera_info</cameraInfoTopicName>
-            <frameName>camera_link</frameName>
-            <hackBaseline>0.07</hackBaseline>
-            <distortionK1>0.0</distortionK1>
-            <distortionK2>0.0</distortionK2>
-            <distortionK3>0.0</distortionK3>
-            <distortionT1>0.0</distortionT1>
-            <distortionT2>0.0</distortionT2>
-          </plugin>
+          <topic>camera/image_raw</topic>
+          <gz_frame_id>camera_link_optical</gz_frame_id>
         </sensor>
   </gazebo> -->

Commit message: fixes

File: revolt_description/urdf/revolt.urdf.xacro (robot description, xacro)
@@ -142,5 +142,5 @@
     <joint name="camera_joint" type="fixed">
         <origin xyz="-0.0065090556831789159187 0.028999999999999984124 1.1221743816224209809e-05"
-            rpy="-1.570796326794896558 3.2526065174728515974e-16 1.570796326794896558" />
+            rpy="1.570796326794896558 3.2526065174728515974e-16 3.141592653589793116" />
         <parent link="camera_mount" />
         <child link="camera_link" />
@@ -188,6 +188,4 @@
         <child link="left_wheel" />
         <axis xyz="0 0 1" />
-        <limit effort="1" velocity="20" />
-        <joint_properties friction="0.0" />
     </joint>
     <!-- ................................ RIGHT WHEEL .................................. -->
@@ -223,6 +221,4 @@
         <child link="right_wheel" />
         <axis xyz="0 0 -1" />
-        <limit effort="1" velocity="20" />
-        <joint_properties friction="0.0" />
     </joint>
     <!-- ................................ FRONT CASTER WHEEL .................................. -->
@@ -298,5 +294,5 @@
         <joint name="frontcaster_rotation_joint" type="continuous">
             <origin
-                xyz="-0.094939000879477097872 -2.5246608566260299064e-10 -0.0082499999999999969191"
+                xyz="-0.094939000879477097872 -2.5246608566260299064e-10 -0.0075"
                 rpy="0 -0 -3.141592653589793116" />
             <parent link="chassis" />
@@ -325,5 +321,7 @@
         </inertial>
     </link>
-    <link name="caster_wheel_2">
+    <link name="caster_wheel_2"><limit>
+      <effort>20</effort> <!-- from <wheel_torque> in libgazebo_ros_diff_drive.so.-->
+    </limit>
         <visual>
             <origin xyz="0 0 8.6736173798840354721e-19"
@@ -379,5 +377,5 @@
         <joint name="backcaster_rotation_joint" type="continuous">
             <origin
-                xyz="0.097009446841797339345 -2.4932854392201164728e-10 -0.0082499999999999969191"
+                xyz="0.097009446841797339345 -2.4932854392201164728e-10 -0.0075"
                 rpy="0 -0 1.3216940769347106485e-16" />
             <parent link="chassis" />

File: revolt_gazebosim/urdf/revolt_gazebosim.xacro (robot description, xacro)
@@ -3,19 +3,7 @@
   <xacro:include filename="$(find revolt_description)/urdf/revolt.urdf.xacro"/>
 	  <gazebo>
-    <!-- <plugin name="revolt_joint_state" filename="libgazebo_ros_joint_state_publisher.so">
-      <ros>
-        <remapping>~/out:=joint_states</remapping>
-        <remapping>/tf:=tf</remapping>
-      </ros>
-      <update_rate>30</update_rate>
-      <joint_name>right_wheel_joint</joint_name>
-      <joint_name>left_wheel_joint</joint_name>
-      <joint_name>frontcaster_rotation_joint</joint_name>
-      <joint_name>frontcaster_wheel_joint</joint_name>
-      <joint_name>backcaster_rotation_joint</joint_name>
-      <joint_name>backcaster_wheel_joint</joint_name>
-    </plugin> -->
     <plugin filename="gz-sim-joint-state-publisher-system" name="gz::sim::systems::JointStatePublisher">
       <topic>joint_states</topic> <!--from <ros><remapping> -->
+      <update_rate>5</update_rate>
       <joint_name>right_wheel_joint</joint_name>
       <joint_name>left_wheel_joint</joint_name>
@@ -33,5 +21,5 @@
       <wheel_radius>0.038</wheel_radius>
       <!-- limits -->
-      <max_linear_acceleration>0.033</max_linear_acceleration> <!-- computed from <max_linear_acceleration> in the original plugin-->
+      <max_linear_acceleration>1</max_linear_acceleration> <!-- computed from <max_linear_acceleration> in the original plugin-->
       <topic>cmd_vel</topic> <!-- from <commant_topic> -->
       <odom_topic>odom</odom_topic> <!-- from <odometry_topic> -->
@@ -42,28 +30,4 @@
     </plugin>
 	  </gazebo>
-<!--
-    <gazebo reference="rplidar_laser_link">
-      <sensor name="laser" type="gpu_lidar">
-        <visualize>false</visualize>
-        <update_rate>10</update_rate>
-        <lidar>
-          <scan>
-            <horizontal>
-            <samples>720</samples>
-            <resolution>1</resolution>
-            <min_angle>-3.14</min_angle>
-            <max_angle>3.14</max_angle>
-            </horizontal>
-          </scan>
-          <range>
-            <min>0.10</min>
-            <max>12.0</max>
-            <resolution>0.01</resolution>
-          </range>
-        </lidar>
-        <topic>scan</topic>
-        <gz_frame_id>rplidar_laser_link</gz_frame_id>
-      </sensor>
-    </gazebo> -->
     <gazebo reference="rplidar_laser_link">
         <sensor name="gpu_lidar" type="gpu_lidar">
@@ -95,33 +59,5 @@
         </sensor>
     </gazebo>
-        <!-- <sensor name="gpu_lidar" type="gpu_lidar">
-          <always_on>true</always_on>
-          <visualize>true</visualize>
-          <pose>-0.064 0 0.121 0 0 0</pose>
-          <update_rate>5</update_rate>
-          <topic>scan</topic>
-          <gz_frame_id>base_scan</gz_frame_id>
-          <lidar>
-              <scan>
-                  <horizontal>
-                      <samples>360</samples>
-                      <resolution>1</resolution>
-                      <min_angle>-3.14</min_angle>
-                      <max_angle>3.14</max_angle>
-                  </horizontal>
-              </scan>
-              <range>
-                  <min>0.10</min>
-                  <max>12.0</max>
-                  <resolution>0.01</resolution>
-              </range>
-              <noise>
-                  <type>gaussian</type>
-                  <mean>0.0</mean>
-                  <stddev>0.001</stddev>
-              </noise>
-          </lidar>
-        </sensor> -->
-    <!-- <joint name="camera_optical_joint" type="fixed">
+    <joint name="camera_optical_joint" type="fixed">
         <parent link="camera_link"/>
         <child link="camera_link_optical"/>
@@ -133,5 +69,6 @@
         <sensor name='camera' type='camera'>
           <camera>
-            <horizontal_fov>1.047</horizontal_fov>
+            <camera_info_topic>camera/camera_info</camera_info_topic>
+            <horizontal_fov>1.089</horizontal_fov>
             <image>
               <width>640</width>
@@ -139,13 +76,13 @@
             </image>
             <clip>
-              <near>0.1</near>
-              <far>100</far>
+              <near>0.05</near>
+              <far>8.0</far>
             </clip>
           </camera>
-          <always_on>1</always_on>
-          <update_rate>30</update_rate>
-          <topic>camera/image_raw</topic>
+          <update_rate>10</update_rate>
+          <visualize>true</visualize>
+          <topic>camera/image_raw</topic>`
           <gz_frame_id>camera_link_optical</gz_frame_id>
         </sensor>
-  </gazebo> -->
+  </gazebo>
 </robot>

Commit message: Added gz playground

File: revolt_description/urdf/revolt.urdf.xacro (robot description, xacro)
@@ -148,10 +148,10 @@
     </joint>
     <!-- ................................ LIDAR .................................. -->
-    <link name="rplidar_laser_link" />
+    <link name="rplidar_laser" />
     <joint name="rplidar_laser_joint" type="fixed">
         <origin xyz="0.068995117891150689604 0.00011464698805746520449 0.15024683531486093813"
             rpy="0 0 ${pi}" />
         <parent link="chassis" />
-        <child link="rplidar_laser_link" />
+        <child link="rplidar_laser" />
         <axis xyz="0 0 0" />
     </joint>
@@ -321,7 +321,8 @@
         </inertial>
     </link>
-    <link name="caster_wheel_2"><limit>
-      <effort>20</effort> <!-- from <wheel_torque> in libgazebo_ros_diff_drive.so.-->
-    </limit>
+    <link name="caster_wheel_2">
+        <!-- <limit>
+      <effort>20</effort>
+    </limit> -->
         <visual>
             <origin xyz="0 0 8.6736173798840354721e-19"

File: revolt_gazebosim/urdf/revolt_gazebosim.xacro (robot description, xacro)
@@ -30,5 +30,5 @@
     </plugin>
 	  </gazebo>
-    <gazebo reference="rplidar_laser_link">
+    <gazebo reference="rplidar_laser">
         <sensor name="gpu_lidar" type="gpu_lidar">
           <always_on>true</always_on>
@@ -36,5 +36,5 @@
           <update_rate>5</update_rate>
           <topic>scan</topic>
-          <gz_frame_id>base_scan</gz_frame_id>
+          <gz_frame_id>rplidar_laser</gz_frame_id>
           <lidar>
               <scan>

Commit message: Added SLAM package

File: revolt_description/urdf/revolt.urdf.xacro (robot description, xacro)
@@ -322,7 +322,4 @@
     </link>
     <link name="caster_wheel_2">
-        <!-- <limit>
-      <effort>20</effort>
-    </limit> -->
         <visual>
             <origin xyz="0 0 8.6736173798840354721e-19"

File: revolt_gazebosim/urdf/revolt_gazebosim.xacro (robot description, xacro)
@@ -59,4 +59,13 @@
         </sensor>
     </gazebo>
+    <gazebo reference="imu_frame">
+      <sensor name="imu_sensor" type="imu">
+          <always_on>1</always_on>
+          <update_rate>1</update_rate>
+          <gz_frame_id>imu_frame</gz_frame_id>
+          <visualize>true</visualize>
+          <topic>imu</topic>
+      </sensor>
+    </gazebo>
     <joint name="camera_optical_joint" type="fixed">
         <parent link="camera_link"/>
